Commit message: halfway through keyboard_control_arm

File: 2_keyboard_control_arm/keyboard_control_arm/urdf/beam_balance.urdf (robot description, URDF)
Before this commit: robot movable_arm, 3 links, 2 joints
Links:
- added link shoulder_link, mass 5; collision cylinder length=0.6 radius=0.3; visual cylinder length=0.6 radius=0.3
- added link world
- link base_link: mass 1 -> 20
- link beam_link_1: mass 1 -> 5; geometry collision box size=0.3 0.3 7; visual box size=0.3 0.3 7
- link beam_link_2: geometry collision box size=0.3 0.3 7; visual box size=0.3 0.3 7
Joints:
- removed joint base_to_beam
- added joint base_to_shoulder: type continuous, parent base_link, child shoulder_link, origin xyz=0 0 1.7 rpy=0 0 0
- added joint fixed: type fixed, parent world, child base_link
- added joint shoulder_to_beam1: type continuous, parent shoulder_link, child beam_link_1, origin xyz=0 0 0 rpy=1 0 0, axis 1 0 0
- joint beam_1_to_beam_2: origin (none) -> xyz=0.3 0 3.5 rpy=0 0 0.785

Commit message: lesson 2 files

File: 2_keyboard_control_arm/keyboard_control_arm/urdf/beam_balance.urdf (robot description, URDF)
Before this commit: robot movable_arm, 5 links, 4 joints
Joints:
- joint base_to_shoulder: limit (none) -> lower=0 upper=0 effort=1000.0 velocity=0.5; type continuous -> revolute
- joint shoulder_to_beam1: axis 1 0 0 -> -1 0 0; origin xyz=0 0 0 rpy=1 0 0 -> xyz=0 0 0 rpy=-1.57075 0 0

File: 2_keyboard_control_arm/keyboard_control_arm/urdf/sphere.urdf (robot description, URDF)
Before this commit: robot myfirst, 1 links, 0 joints
Links:
- link base_link: mass 1 -> 10; geometry collision sphere radius=0.2; visual sphere radius=0.2
